Commit message: change lidar orientation

File: diffbot_control/description/lidar.xacro (robot description, xacro)
@@ -9,5 +9,5 @@
                 <parent link="chassis" />
                 <child link="lidar_frame" />
-                <origin xyz="${-lidar_radius} 0 ${chassis_height}" rpy="0 0 0" />
+                <origin xyz="${-lidar_radius} 0 ${chassis_height}" rpy="${pi} ${pi} 0" />
         </joint>
         <link name="lidar_frame">
