Commit message: can now do sim and real

File: diffbot_control/description/robot.urdf.xacro (robot description, xacro)
@@ -1,4 +1,5 @@
 <?xml version="1.0"?>
 <robot xmlns:xacro="http://www.ros.org/wiki/xacro"  name="my_robot">
+        <xacro:arg name="sim_mode" default="false"/>
         <xacro:include filename="robot_real.xacro"/>
         <!-- <xacro:include filename="robot_core.xacro" /> -->

File: diffbot_control/description/ros2_control.xacro (robot description, xacro)
@@ -1,49 +1,54 @@
 <?xml version="1.0"?>
 <robot xmlns:xacro="http://www.ros.org/wiki/xacro">
-        <!-- <ros2_control name="GazeboSystem" type="system">
-                <hardware>
-                        <plugin>gz_ros2_control/GazeboSimSystem</plugin>
-                </hardware>
-                <joint name="left_wheel_joint">
-                        <command_interface name="velocity">
-                                <param name="min">-5</param>
-                                <param name="max">5</param>
-                        </command_interface>
-                        <state_interface name="velocity"/>
-                        <state_interface name="position"/>
-                </joint>
-                <joint name="right_wheel_joint">
-                        <command_interface name="velocity">
-                                <param name="min">-5</param>
-                                <param name="max">5</param>
-                        </command_interface>
-                        <state_interface name="velocity"/>
-                        <state_interface name="position"/>
-                </joint>
-        </ros2_control> -->
-        <ros2_control name="RealRobot" type="system">
-                <hardware>
-                        <plugin>diffbot_system_hw/DiffBotSystemHardware</plugin>
-                        <param name="left_wheel_name">left_wheel_joint</param>
-                        <param name="right_wheel_name">right_wheel_joint</param>
-                        <param name="angle_resolution">0.001534</param>
-                        <param name="encoder_counts_per_rev">4096</param>
-                        <param name="cmd_vel_diff_threshold">0.07</param>
-                </hardware>
-                <joint name="left_wheel_joint">
-                        <command_interface name="velocity"/>
-                        <state_interface name="position" />
-                        <state_interface name="velocity" />
-                </joint>
-                <joint name="right_wheel_joint">
-                        <command_interface name="velocity"/>
-                        <state_interface name="position" />
-                        <state_interface name="velocity" />
-                </joint>
-        </ros2_control>
+        <xacro:if value="$(arg sim_mode)">
+                <ros2_control name="GazeboSystem" type="system">
+                        <hardware>
+                                <plugin>gz_ros2_control/GazeboSimSystem</plugin>
+                        </hardware>
+                        <joint name="left_wheel_joint">
+                                <command_interface name="velocity">
+                                        <param name="min">-5</param>
+                                        <param name="max">5</param>
+                                </command_interface>
+                                <state_interface name="velocity" />
+                                <state_interface name="position" />
+                        </joint>
+                        <joint name="right_wheel_joint">
+                                <command_interface name="velocity">
+                                        <param name="min">-5</param>
+                                        <param name="max">5</param>
+                                </command_interface>
+                                <state_interface name="velocity" />
+                                <state_interface name="position" />
+                        </joint>
+                </ros2_control>
+        </xacro:if>
+        <xacro:unless value="$(arg sim_mode)">
+                <ros2_control name="RealRobot" type="system">
+                        <hardware>
+                                <plugin>diffbot_system_hw/DiffBotSystemHardware</plugin>
+                                <param name="left_wheel_name">left_wheel_joint</param>
+                                <param name="right_wheel_name">right_wheel_joint</param>
+                                <param name="angle_resolution">0.001534</param>
+                                <param name="encoder_counts_per_rev">4096</param>
+                                <param name="cmd_vel_diff_threshold">0.07</param>
+                        </hardware>
+                        <joint name="left_wheel_joint">
+                                <command_interface name="velocity"/>
+                                <state_interface name="position" />
+                                <state_interface name="velocity" />
+                        </joint>
+                        <joint name="right_wheel_joint">
+                                <command_interface name="velocity"/>
+                                <state_interface name="position" />
+                                <state_interface name="velocity" />
+                        </joint>
+                </ros2_control>
+        </xacro:unless>
         <gazebo>
                 <plugin name="gz_ros2_control::GazeboSimROS2ControlPlugin"
                         filename="libgz_ros2_control-system.so">
                         <parameters>$(find diffbot_control)/config/ros2_controllers.yaml</parameters>
+                        <parameters>$(find diffbot_control)/config/gazebo_ros2_controllers.yaml</parameters>
                 </plugin>
         </gazebo>
